Commit message: 修复ROS2运行bug,验证图灵6轴ROS2控制代码

File: src/mercury_robot_urdf/mercury_robot_urdf/urdf/mercury_x1/mercury_x1.urdf (robot description, URDF)
Before this commit: robot firefighter, 18 links, 18 joints
Links:
- added link base_footprint

File: src/mercury_robot_urdf/mercury_robot_urdf/urdf/mercury_x1/mercury_x1_turing_stack.urdf (robot description, URDF)
Before this commit: robot firefighter, 18 links, 18 joints
Links:
- added link base_footprint
