Commit message: 增加水星图灵6轴机械臂ROS2控制代码

File: src/mercury_robot_urdf/mercury_robot_urdf/urdf/mercury_x1/mercury_x1_turing_stack.urdf (robot description, URDF)
Before this commit: robot firefighter, 18 links, 18 joints
Joints:
- removed joint joint7_L
- removed joint joint7_R
- added joint joint3_L_hide: type fixed, parent link2_L, child link3_L, origin xyz= 0 -0.11 0   rpy=1.5708 0 0, axis  0 0 1, limit lower=-2.879 upper=2.879 effort=1000.0 velocity=0
- added joint joint3_R_hide: type fixed, parent link2_R, child link3_R, origin xyz= 0 -0.11 0   rpy=1.5708 0 0, axis  0 0 1, limit lower=-2.879 upper=2.879 effort=1000.0 velocity=0
- joint body: type revolute -> fixed
- joint eye: limit lower=0 upper=0.83 effort=1000.0 velocity=0 -> lower=-1.04 upper=0 effort=1000.0 velocity=0
- joint head: limit lower=-2.4085 upper=3.2812 effort=1000.0 velocity=0 -> lower=-2.321 upper=3.2812 effort=1000.0 velocity=0
- joint joint3_L: child link3_L -> link4_L; limit lower=-2.879 upper=2.879 effort=1000.0 velocity=0 -> lower=-2.879 upper=0.087 effort=1000.0 velocity=0; origin xyz= 0 -0.11 0   rpy=1.5708 0 0 -> xyz= 0.03 0 0.095 rpy=-1.5708 0 3.14159; parent link2_L -> link3_L
- joint joint3_R: child link3_R -> link4_R; limit lower=-2.879 upper=2.879 effort=1000.0 velocity=0 -> lower=-2.879 upper=0.087 effort=1000.0 velocity=0; origin xyz= 0 -0.11 0   rpy=1.5708 0 0 -> xyz= 0.03 0 0.095 rpy=-1.5708 0 3.14159; parent link2_R -> link3_R
- joint joint4_L: child link4_L -> link5_L; limit lower=-2.879 upper=0.087 effort=1000.0 velocity=0 -> lower=-2.879 upper=2.879 effort=1000.0 velocity=0; origin xyz= 0.03 0 0.095 rpy=-1.5708 0 3.14159 -> xyz= 0.03 -0.126 0 rpy=1.5708 3.14159 0; parent link3_L -> link4_L
- joint joint4_R: child link4_R -> link5_R; limit lower=-2.879 upper=0.087 effort=1000.0 velocity=0 -> lower=-2.879 upper=2.879 effort=1000.0 velocity=0; origin xyz= 0.03 0 0.095 rpy=-1.5708 0 3.14159 -> xyz= 0.03 -0.126 0 rpy=1.5708 3.14159 0; parent link3_R -> link4_R
- joint joint5_L: child link5_L -> link6_L; limit lower=-2.879 upper=2.879 effort=1000.0 velocity=0 -> lower=-1.9198 upper=3.0543 effort=1000.0 velocity=0; origin xyz= 0.03 -0.126 0 rpy=1.5708 3.14159 0 -> xyz= 0 0 0.08 rpy=1.5708 -1.5708 0; parent link4_L -> link5_L
- joint joint5_R: child link5_R -> link6_R; limit lower=-2.879 upper=2.879 effort=1000.0 velocity=0 -> lower=-1.9198 upper=3.0543 effort=1000.0 velocity=0; origin xyz= 0.03 -0.126 0 rpy=1.5708 3.14159 0 -> xyz= 0 0 0.08 rpy=1.5708 -1.5708 0; parent link4_R -> link5_R
- joint joint6_L: child link6_L -> link7_L; limit lower=-1.9198 upper=3.0543 effort=1000.0 velocity=0 -> lower=-3.14 upper=3.14 effort=1000.0 velocity=0; origin xyz= 0 0 0.08 rpy=1.5708 -1.5708 0 -> xyz= 0.038 -0.046 0 rpy=1.5708 0 0; parent link5_L -> link6_L
- joint joint6_R: child link6_R -> link7_R; limit lower=-1.9198 upper=3.0543 effort=1000.0 velocity=0 -> lower=-3.14 upper=3.14 effort=1000.0 velocity=0; origin xyz= 0 0 0.08 rpy=1.5708 -1.5708 0 -> xyz= 0.038 -0.046 0 rpy=1.5708 0 0; parent link5_R -> link6_R

Commit message: feat(Turing X1-URDF): Add two left and right camera models to the urdf model head and update the coordinate axis

File: src/mercury_robot_urdf/mercury_robot_urdf/urdf/mercury_x1/mercury_x1_turing_stack.urdf (robot description, URDF)
Before this commit: robot firefighter, 19 links, 18 joints
Links:
- added link link_left_camera, mass 0; collision mesh filename=package://mercury_robot_urdf/urdf/mercury_x1/left_camera.dae; visual mesh filename=package://mercury_robot_urdf/urdf/mercury_x1/left_camera.dae
- added link link_right_camera, mass 0; collision mesh filename=package://mercury_robot_urdf/urdf/mercury_x1/right_camera.d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; visual mesh filename=package://mercury_robot_urdf/urdf/mercury_x1/right_camera.d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
- link base_link: mass None -> 47.2640
- link link1_L: mass None -> 0.784
- link link1_R: mass None -> 0.784
- link link2_L: mass None -> 0
- link link2_R: mass None -> 0
- link link3_L: mass None -> 0.824
- link link3_R: mass None -> 0.824
- link link4_L: mass None -> 0.7
- link link4_R: mass None -> 0.7
- link link5_L: mass None -> 0.508
- link link5_R: mass None -> 0.508
- link link6_L: mass None -> 0.398
- link link6_R: mass None -> 0.398
- link link7_L: mass None -> 0.393
- link link7_R: mass None -> 0.393
- link link_body: mass None -> 5.516
- link link_eye: mass None -> 0; geometry collision mesh filename=package://mercury_robot_urdf/urdf/mercury_x1/dual_hole_came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; visual mesh filename=package://mercury_robot_urdf/urdf/mercury_x1/dual_hole_came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
- link link_head: mass None -> 0
Joints:
- added joint left_camera: type fixed, parent link_eye, child link_left_camera, origin xyz= 0.008 0 -0.027  rpy=0 0 0, axis  0 0 1, limit lower=-1.04 upper=0 effort=1000.0 velocity=0
- added joint right_camera: type fixed, parent link_eye, child link_right_camera, origin xyz= 0.008 0 0.033  rpy=0 0 0, axis  0 0 1, limit lower=-1.04 upper=0 effort=1000.0 velocity=0
